File: ecad/carrier/carrier.kicad_sch (KiCad schematic)
At the start: 121 parts, among them J1 XT30PW-M battery, J10 Servo chain 2, J11 Servo chain 3, J12 Servo chain 3, J13 Speaker CMS-18132-18SP, J14 Head board, J2 Cell sense: MID, NTC, J3 Main switch, J4 USB-C charge, J5 Radxa ZERO 3W, J6 Debug UART, J7 Servo chain 1, J8 Servo chain 1, J9 Servo chain 2, U1 TPS259824LNRGE, U10 MAX98357AETE+T, U11 BNO085, U2 TPS56C215RNNR, U3 TPS62933DRLR, U4 TLV75533PDBVR, U5 BQ25887RGER, U6 ADS1115IDGSR, U7 74LVC2G241DCUR, U8 74LVC2G241DCUR, U9 74LVC2G241DCUR

Commit message: Phase 2 complete: carrier board PCB, harness, DCK-02 rev A
- Generated 4-layer 76 x 62 mm carrier PCB: placement, Freerouting, power
  pours and stitching; DRC 0 violations, 0 unconnected, 0 parity issues
- STEP export for Fusion, renders, end-to-end build script
- Harness definition from params.py with service loops per joint travel
- Asset register, CLAUDE.md and README updated; head board deferred (RK9)

Co-Authored-By: Claude Opus 5.5 <noreply@anthropic.com>
Parts:
- H1, H2, H3, H4: now left out of the parts list
Changed lines of the file:
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@@
 		(unit 1)
 		(exclude_from_sim no)
-		(in_bom yes)
+		(in_bom no)
 		(on_board yes)
 		(dnp no)
@@
 		(unit 1)
 		(exclude_from_sim no)
-		(in_bom yes)
+		(in_bom no)
 		(on_board yes)
 		(dnp no)
@@
 		(unit 1)
 		(exclude_from_sim no)
-		(in_bom yes)
+		(in_bom no)
 		(on_board yes)
 		(dnp no)
@@
 		(unit 1)
 		(exclude_from_sim no)
-		(in_bom yes)
+		(in_bom no)
 		(on_board yes)
 		(dnp no)
